File: TEC Driver 50W/TEC Driver 50W.kicad_pcb (KiCad board)
At the start: 2 copper layers, 15 parts, among them U1 SC8903

Commit message: 04/18
Parts:
- removed C12: 220u, 35V, AEX7 MOS:Cap_Al_D6.3xH11.5mm_Hor
- added C13: 15n, Capacitor_SMD:C_0603_1608Metric, F.Cu at (117.0, 65.8)
- added C14: 1u, Capacitor_SMD:C_0603_1608Metric, F.Cu at (119.2, 68.0)
- added C15: 1u, Capacitor_SMD:C_0603_1608Metric, F.Cu at (130.8, 64.2)
- added C16: 220u, 35V, AEX7 MOS:Cap_Al_D6.3xH11.5mm_Hor, F.Cu at (113.2, 77.0)
- added R10: 47k, Resistor_SMD:R_0603_1608Metric, F.Cu at (130.8, 65.8)
- added R11: NC, Resistor_SMD:R_0603_1608Metric, F.Cu at (133.8, 64.2)
- added R12: 200k, Resistor_SMD:R_0603_1608Metric, F.Cu at (133.8, 62.8)
- added R2: 0R, Resistor_SMD:R_0603_1608Metric, F.Cu at (119.2, 63.5)
- added R3: 5mR, Resistor_SMD:R_1206_3216Metric, F.Cu at (127.5, 72.2)
- added R4: 5mR, Resistor_SMD:R_1206_3216Metric, F.Cu at (122.5, 72.2)
- added R5: 47k, Resistor_SMD:R_0603_1608Metric, F.Cu at (119.2, 65.0)
- added R6: 15k, Resistor_SMD:R_0603_1608Metric, F.Cu at (119.2, 66.5)
- added R7: 160k, Resistor_SMD:R_0603_1608Metric, F.Cu at (115.5, 65.8)
- added R8: 9k1, Resistor_SMD:R_0603_1608Metric, F.Cu at (116.2, 68.0)
- added R9: 47k, Resistor_SMD:R_0603_1608Metric, F.Cu at (133.8, 65.8)
- C10, C3, C4, C5, C6, C7, C8, C9: footprint Resistor_SMD:R_1206_3216Metric -> Capacitor_SMD:C_1206_3216Metric
- C11: footprint AEX7 MOS:Cap_Al_D6.3xH11.5mm_Hor -> AEX7 MOS:Cap_Al_D6.3xH11.5mm_Hor_Flip
- moved R1 14.2 mm to (130.8, 68.0), turned to 180 degrees
- moved C7 10.7 mm to (112.2, 71.2), turned to 90 degrees
- moved C6 10.4 mm to (137.8, 71.2), turned to 90 degrees
- moved C10 9.52 mm to (119.0, 71.2), turned to 90 degrees
- moved C3 9.42 mm to (131.0, 71.2), turned to 90 degrees
- moved C8 9.28 mm to (114.5, 71.2), turned to 90 degrees
- moved C5 9.06 mm to (135.5, 71.2), turned to 90 degrees
- moved C9 8.85 mm to (116.8, 71.2), turned to 90 degrees
- moved C4 8.68 mm to (133.2, 71.2), turned to 90 degrees
- moved C11 4.64 mm to (136.8, 77.0), turned to 180 degrees
- moved C2 0.25 mm to (123.2, 61.8)
- moved U1 0.11 mm to (125.0, 66.8)
Connections:
- C10 pad 1: VOUTP -> VOUT
- C11 pad 1: VINP -> VIN
- C3 pad 1: VINP -> VIN
- C4 pad 1: VINP -> VIN
- C5 pad 1: VINP -> VIN
- C6 pad 1: VINP -> VIN
- C7 pad 1: VOUTP -> VOUT
- C8 pad 1: VOUTP -> VOUT
- C9 pad 1: VOUTP -> VOUT
- U1 pad 10: unconnected-(U1-VOUT_SN-Pad10) -> VOUT
- U1 pad 11: unconnected-(U1-VOUT_SP-Pad11) -> VOUTP
- U1 pad 18: unconnected-(U1-VIN_SN-Pad18) -> VINP
- U1 pad 19: unconnected-(U1-VIN_SP-Pad19) -> VIN
- U1 pad 20: Net-(U1-PGND-Pad20) -> GND
- U1 pad 21: unconnected-(U1-/CE-Pad21) -> /~{SC8903_EN}
- U1 pad 23: Net-(U1-PGND-Pad20) -> GND
- U1 pad 24: Net-(U1-PGND-Pad20) -> GND
- U1 pad 25: Net-(U1-PGND-Pad20) -> GND
- U1 pad 26: Net-(U1-PGND-Pad20) -> GND
- U1 pad 27: unconnected-(U1-ILIM_I-Pad27) -> Net-(U1-ILIM_I)
- U1 pad 28: unconnected-(U1-INACT-Pad28) -> /INACT
- U1 pad 29: unconnected-(U1-MODE-Pad29) -> Net-(U1-MODE)
- U1 pad 3: unconnected-(U1-FREQ-Pad3) -> Net-(U1-FREQ)
- U1 pad 30: unconnected-(U1-VCC-Pad30) -> Net-(U1-VCC)
- U1 pad 36: unconnected-(U1-LG-Pad36) -> Net-(U1-LD2)
- U1 pad 38: unconnected-(U1-LD2-Pad38) -> Net-(U1-LD2)
- U1 pad 39: unconnected-(U1-VPWM-Pad39) -> /VPWM
- U1 pad 4: unconnected-(U1-AGND-Pad4) -> GND
- U1 pad 6: unconnected-(U1-ILIM_O-Pad6) -> Net-(U1-ILIM_O)
- U1 pad 7: unconnected-(U1-COMP-Pad7) -> Net-(U1-COMP)
- U1 pad 8: unconnected-(U1-FB-Pad8) -> /FB
Routing:
- net GND: track 0.00 -> 10.8 mm
- net Net-(U1-LD2): track 0.00 -> 6.53 mm
- net VOUT: track 0.00 -> 4.86 mm
- net VINP: track 0.00 -> 3.92 mm
- net VIN: track 0.00 -> 3.87 mm
- net VOUTP: track 0.00 -> 3.55 mm
- net /SW1: track 0.00 -> 2.06 mm
- net /BT2: track 0.00 -> 1.96 mm
- net /VPWM: track 0.00 -> 1.15 mm, vias 0 -> 1
- net /~{SC8903_EN}: track 0.00 -> 0.86 mm, vias 0 -> 1
- added copper zone on F.Cu, net VIN
- added copper zone on F.Cu, net VINP
- added copper zone on F.Cu, net VOUT
- added copper zone on F.Cu, net VOUTP

Commit message: 4/18
Parts:
- added C12: 0u1, Capacitor_SMD:C_0603_1608Metric, F.Cu at (140.8, 68.2)
- added C17: 22p, Capacitor_SMD:C_0603_1608Metric, F.Cu at (105.2, 66.0)
- added C18: 22p, Capacitor_SMD:C_0603_1608Metric, F.Cu at (110.8, 66.0)
- added C19: 100n, Capacitor_SMD:C_0603_1608Metric, F.Cu at (57.0, 81.2)
- added C20: 10u, Capacitor_SMD:C_1206_3216Metric, F.Cu at (138.2, 61.5)
- added C21: 10u, Capacitor_SMD:C_1206_3216Metric, F.Cu at (138.2, 59.2)
- added C22: 100n, Capacitor_SMD:C_0603_1608Metric, F.Cu at (114.5, 54.2)
- added C23: 100n, Capacitor_SMD:C_0603_1608Metric, F.Cu at (106.0, 51.0)
- added C24: 100n, Capacitor_SMD:C_0603_1608Metric, F.Cu at (102.5, 59.5)
- added C25: 100n, Capacitor_SMD:C_0603_1608Metric, F.Cu at (104.8, 63.0)
- added C26: 100n, Capacitor_SMD:C_0603_1608Metric, F.Cu at (110.2, 63.0)
- added C27: 1u, Capacitor_SMD:C_0603_1608Metric, F.Cu at (145.5, 60.5)
- added C28: 100n, Capacitor_SMD:C_0603_1608Metric, F.Cu at (143.2, 55.8)
- added C29: 100n, Capacitor_SMD:C_0603_1608Metric, F.Cu at (113.0, 62.0)
- added C30: 100n, Capacitor_SMD:C_0603_1608Metric, F.Cu at (61.0, 81.2)
- added C31: 20p, Capacitor_SMD:C_0603_1608Metric, F.Cu at (139.8, 52.0)
- added C32: 47u, Capacitor_Tantalum_SMD:CP_EIA-3216-18_Kemet-A_Pad1.58x1.35mm_HandSolder, F.Cu at (143.0, 52.5)
- added C34: 10u, Capacitor_SMD:C_0603_1608Metric, F.Cu at (146.2, 52.0)
- added C35: 10u, Capacitor_SMD:C_0603_1608Metric, F.Cu at (147.8, 52.0)
- added C37: 10u, Capacitor_SMD:C_0603_1608Metric, F.Cu at (134.2, 56.8)
- added C39: 10n, Capacitor_SMD:C_0603_1608Metric, F.Cu at (136.8, 54.0)
- added C40: 10u, Capacitor_SMD:C_0603_1608Metric, F.Cu at (134.2, 51.2)
- added D2: LED0, LED_SMD:LED_0603_1608Metric, F.Cu at (70.3, 69.2)
- added D3: LED1, LED_SMD:LED_0603_1608Metric, F.Cu at (70.3, 71.8)
- added D4: LED2, LED_SMD:LED_0603_1608Metric, F.Cu at (70.3, 74.4)
- added F1: 1206 8A, Fuse:Fuse_1206_3216Metric, F.Cu at (139.8, 75.8)
- added J1: USB_C_Receptacle_USB2.0_16P, Connector_USB:USB_C_Receptacle_Palconn_UTC16-G, F.Cu at (145.8, 75.0)
- added L2: 6u8, Inductor_SMD:L_Sunlord_MWSA0402S, F.Cu at (146.5, 56.5)
- added R13: 1M, Resistor_SMD:R_0603_1608Metric, F.Cu at (142.2, 68.2)
- added R14: 1k, Resistor_SMD:R_0603_1608Metric, F.Cu at (142.5, 60.5)
- added R15: 10k, Resistor_SMD:R_0603_1608Metric, F.Cu at (148.2, 65.5)
- added R16: 330R, Resistor_SMD:R_0603_1608Metric, F.Cu at (57.0, 79.8)
- added R17: 10k, Resistor_SMD:R_0603_1608Metric, F.Cu at (92.4, 82.0)
- added R18: 1k, Resistor_SMD:R_0603_1608Metric, F.Cu at (92.4, 84.5)
- added R19: 10k, Resistor_SMD:R_0603_1608Metric, F.Cu at (92.4, 87.0)
- added R20: 1k, Resistor_SMD:R_0603_1608Metric, F.Cu at (66.9, 61.7)
- added R21: 1k, Resistor_SMD:R_0603_1608Metric, F.Cu at (66.9, 64.2)
- added R22: 1k, Resistor_SMD:R_0603_1608Metric, F.Cu at (66.9, 66.7)
- added R23: 24k, Resistor_SMD:R_0603_1608Metric, F.Cu at (148.2, 62.5)
- added R24: 10k, Resistor_SMD:R_0603_1608Metric, F.Cu at (102.5, 56.5)
- added R25: 10k, Resistor_SMD:R_0603_1608Metric, F.Cu at (113.0, 65.0)
- added R26: 330R, Resistor_SMD:R_0603_1608Metric, F.Cu at (61.0, 79.8)
- added R27: 1k, Resistor_SMD:R_0603_1608Metric, F.Cu at (92.4, 89.5)
- added R28: 54k6, Resistor_SMD:R_0603_1608Metric, F.Cu at (138.2, 52.0)
- added R29: 10k, Resistor_SMD:R_0603_1608Metric, F.Cu at (138.2, 55.0)
- added SW1: BTN, Button_Switch_SMD:SW_SPST_PTS810, F.Cu at (57.0, 76.0)
- added SW5: BTN, Button_Switch_SMD:SW_SPST_PTS810, F.Cu at (61.0, 76.0)
- added U2: STM32F103C8Tx, Package_QFP:LQFP-48_7x7mm_P0.5mm, F.Cu at (108.5, 57.0)
- added U3: CH224K, AEX7 Others:ESSOP-10_3.9x4.9mm_P1.00mm, F.Cu at (144.0, 64.0)
- added U4: RY8411, Package_TO_SOT_SMD:SOT-23-6, F.Cu at (140.8, 55.8)
- added U5: RS3236, Package_TO_SOT_SMD:SOT-23-5, F.Cu at (134.2, 54.0)
- added Y2: 8Mhz, Crystal:Crystal_SMD_3225-4Pin_3.2x2.5mm, F.Cu at (108.0, 66.0)
- moved R12 18.7 mm to (115.8, 57.8)
- moved R10 16.7 mm to (115.2, 59.5), turned to -90 degrees
- moved R11 3.09 mm to (130.8, 65.0)
- moved R9 1.68 mm to (133.0, 64.2), turned to 90 degrees
- moved R2 1.50 mm to (117.8, 63.5)
- moved R5 1.06 mm to (118.5, 65.8), turned to 90 degrees
- moved R6 1.06 mm to (120.0, 65.8), turned to 90 degrees
- moved C15 0.75 mm to (130.8, 63.5)
- moved L1 0.50 mm to (124.5, 55.8)
Connections:
- R1 pad 1: VINP -> VIN
Routing:
- net VIN: track 3.87 -> 60.0 mm, vias 0 -> 4
- net Net-(U3-DP): track 0.00 -> 17.2 mm
- net /INACT: track 0.00 -> 16.9 mm, vias 0 -> 2
- net Net-(U3-DM): track 0.00 -> 14.8 mm
- net Net-(J1-CC1): track 0.00 -> 14.2 mm
- net VOUT: track 4.86 -> 17.4 mm
- net +5V: track 0.00 -> 11.6 mm, vias 0 -> 3
- net Net-(J1-CC2): track 0.00 -> 10.3 mm, vias 0 -> 2
- net Net-(F1-Pad1): track 0.00 -> 7.91 mm
- net Net-(U1-ILIM_I): track 0.00 -> 5.25 mm
- net Net-(U4-FB): track 0.00 -> 4.51 mm
- net Net-(U1-FREQ): track 0.00 -> 4.37 mm
- net GND: track 10.8 -> 6.54 mm, vias 0 -> 51
- net Net-(U3-VDD): track 0.00 -> 3.90 mm
- net /VPWM: track 1.15 -> 4.92 mm, vias 1 -> 2
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- added copper zone on F.Cu, net +5V
- added copper zone on B.Cu, net /SW1
- added copper zone on F.Cu, net /SW1
- added copper zone on B.Cu, net /SW2
- added copper zone on F.Cu, net /SW2
- added copper zone on F.Cu, net Net-(U4-LX)
Other:
- board outline added: 50 x 36 mm
