File: TEC Driver 50W/TEC Driver 50W.kicad_sch (KiCad schematic)
At the start: 15 parts, among them U1 SC8903

Commit message: 04/18
Parts:
- removed C12: 220u, 35V, AEX7 MOS:Cap_Al_D6.3xH11.5mm_Hor, symbol Device:C_Polarized
- added C12: 0u1, Capacitor_SMD:C_0603_1608Metric, symbol Device:C_Small
- added C13: 15n, Capacitor_SMD:C_0603_1608Metric, symbol Device:C_Small
- added C14, C15, C27: 1u, Capacitor_SMD:C_0603_1608Metric, symbol Device:C_Small
- added C16: 220u, 35V, AEX7 MOS:Cap_Al_D6.3xH11.5mm_Hor, symbol Device:C_Polarized
- added C17, C18: 22p, Capacitor_SMD:C_0603_1608Metric, symbol Device:C_Small
- added C19, C20, C22, C23, C24, C25, C26: 100n, Capacitor_SMD:C_0603_1608Metric, symbol Device:C_Small
- added C21: 4.7u, Capacitor_SMD:C_0603_1608Metric, symbol Device:C_Small
- added D2: LED0, LED_SMD:LED_0603_1608Metric, symbol Device:LED
- added D3: LED1, LED_SMD:LED_0603_1608Metric, symbol Device:LED
- added D4: LED2, LED_SMD:LED_0603_1608Metric, symbol Device:LED
- added F1: 1206 8A, Fuse:Fuse_1206_3216Metric, symbol Device:Polyfuse_Small
- added J1: USB_C_Receptacle_USB2.0_16P, symbol Connector:USB_C_Receptacle_USB2.0_16P
- added R10, R13, R5, R9: 47k, Resistor_SMD:R_0603_1608Metric, symbol Device:R_Small
- added R11: NC, Resistor_SMD:R_0603_1608Metric, symbol Device:R_Small
- added R12: 200k, Resistor_SMD:R_0603_1608Metric, symbol Device:R_Small
- added R14, R20, R21, R22: 1k, Resistor_SMD:R_0603_1608Metric, symbol Device:R_Small
- added R15, R18, R19: 10k, Resistor_SMD:R_0603_1608Metric, symbol Device:R_Small
- added R16, R17: 330R, Resistor_SMD:R_0603_1608Metric, symbol Device:R_Small
- added R2: 0R, Resistor_SMD:R_0603_1608Metric, symbol Device:R_Small
- added R23: 24k, Resistor_SMD:R_0603_1608Metric, symbol Device:R_Small
- added R3, R4: 5mR, Resistor_SMD:R_1206_3216Metric, symbol Device:R_Small_US
- added R6: 15k, Resistor_SMD:R_0603_1608Metric, symbol Device:R_Small
- added R7: 160k, Resistor_SMD:R_0603_1608Metric, symbol Device:R_Small
- added R8: 9k1, Resistor_SMD:R_0603_1608Metric, symbol Device:R_Small
- added SW1: RST, Button_Switch_SMD:SW_SPST_TL3342, symbol Switch:SW_Push
- added SW2: BOOT0, Button_Switch_SMD:SW_SPST_TL3342, symbol Switch:SW_Push
- added U2: STM32F103C8Tx, Package_QFP:LQFP-48_7x7mm_P0.5mm, symbol MCU_ST_STM32F1:STM32F103C8Tx
- added U3: CH224K, AEX7 Others:ESSOP-10_3.9x4.9mm_P1.00mm, symbol AEX7 Others:CH224
- added Y1: 8Mhz, Crystal:Crystal_SMD_5032-2Pin_5.0x3.2mm, symbol Device:Crystal_Small
- C10, C3, C4, C5, C6, C7, C8, C9: footprint Resistor_SMD:R_1206_3216Metric -> Capacitor_SMD:C_1206_3216Metric
- C11: footprint AEX7 MOS:Cap_Al_D6.3xH11.5mm_Hor -> AEX7 MOS:Cap_Al_D6.3xH11.5mm_Hor_Flip
Connections:
- net GND: now also U1.20 (PGND), U1.23 (PGND), U1.24 (PGND), U1.25 (PGND), U1.26 (PGND), U1.4 (AGND), C12.2, C13.2, C14.2, C15.2, C16.2, C17.1, C18.1, C19.2, C20.2, C21.2, C22.2, C23.2, C24.2, C25.2, C26.2, C27.2, J1.A1 (GND), J1.A12 (GND), J1.B1 (GND), J1.B12 (GND), R11.2, R12.2, R13.2, R19.2, R2.2, R20.2, R21.2, R22.2, R23.2, R5.2, R8.2, R9.2, SW1.2, U2.23 (VSS), U2.35 (VSS), U2.47 (VSS), U2.8 (VSSA), U3.11 (GND)
- net VINP: now also U1.18 (VIN_SN), R3.2; no longer C11.1, C3.1, C4.1, C5.1, C6.1
- net VOUTP: now also U1.11 (VOUT_SP), C14.1, R4.1; no longer C10.1, C7.1, C8.1, C9.1
- net VOUT: now reaches U1.10 (VOUT_SN)
- net VOUT: now also C10.1, C7.1, C8.1, C9.1, C16.1, R4.2, R7.1
- net VIN: now reaches U1.19 (VIN_SP)
- net VIN: now also C11.1, C3.1, C4.1, C5.1, C6.1, F1.2, R14.1, R15.1, R3.1
- net ~{SC8903_EN}: now reaches U1.21 (/CE)
- net at U1.27 (ILIM_I): now also R9.1
- net INACT: now reaches U1.28 (INACT)
- net INACT: now also R10.2
- net at U1.29 (MODE): now also R11.1
- net at U1.3 (FREQ): now also R2.1
- net at U1.30 (VCC): now also C15.1
- net at U1.36 (LG): now also U1.38 (LD2)
- net VPWM: now reaches U1.39 (VPWM)
- net VPWM: now also R12.1
- net at U1.6 (ILIM_O): now also R5.1
- net at U1.7 (COMP): now also R6.1
- net FB: now reaches U1.8 (FB)
- net FB: now also R7.2, R8.1
- new net: C27.1, R14.2, U3.1 (VDD)
- new net: F1.1, J1.A4 (VBUS), J1.A9 (VBUS), J1.B4 (VBUS), J1.B9 (VBUS)
- new net: J1.A5 (CC1), U3.7 (CC1)
- new net: J1.A6 (D+), J1.B6 (D+), U3.4 (DP)
- new net: J1.A7 (D-), J1.B7 (D-), U3.5 (DM)
- new net: J1.B5 (CC2), U3.6 (CC2)
- new net: C12.1, J1.S1 (SHIELD), R13.1
- new net: R23.1, U3.9 (CFG1)
- new net: C17.2, U2.5 (PD0), Y1.1
- new net: C18.2, U2.6 (PD1), Y1.2
- new net: R17.2, R19.1, SW2.2
- new net: D2.1 (K), R20.1
- new net: R16.2, R18.2, SW1.1
- new net: D4.1 (K), R22.1
- new net: D3.1 (K), R21.1
- new net: C13.1, R6.2
- new net: R15.2, U3.8 (VBUS)
- new net +3.3V: C21.1, C22.1, C23.1, C24.1, C25.1, C26.1, R18.1, SW2.1, U2.1 (VBAT), U2.24 (VDD), U2.36 (VDD), U2.48 (VDD), U2.9 (VDDA)
- new net +3V3: R10.1
- new net BOOT0: C20.1, R17.1, U2.44 (BOOT0)
- new net CAN_RX: U2.32 (PA11)
- new net CAN_TX: U2.33 (PA12)
- new net I2C1_SCL: U2.42 (PB6)
- new net I2C1_SDA: U2.43 (PB7)
- new net NRST: C19.1, R16.1, U2.7 (NRST)
- new net PA0_GPIO: U2.10 (PA0)
- new net PA15_GPIO: U2.38 (PA15)
- new net PA1_GPIO: U2.11 (PA1)
- new net PA4_GPIO: U2.14 (PA4)
- new net PA5_GPIO: U2.15 (PA5)
- new net PA6_GPIO: U2.16 (PA6)
- new net PA7_GPIO: U2.17 (PA7)
- new net PA8_BUZZER: U2.29 (PA8)
- new net PB0_LED0: D2.2 (A), U2.18 (PB0)
- new net PB12_GPIO: U2.25 (PB12)
- new net PB13_GPIO: U2.26 (PB13)
- new net PB14_GPIO: U2.27 (PB14)
- new net PB15_GPIO: U2.28 (PB15)
- new net PB1_LED1: D3.2 (A), U2.19 (PB1)
- new net PB2_LED2: D4.2 (A), U2.20 (PB2)
- new net PB3_GPIO: U2.39 (PB3)
- new net PB4_GPIO: U2.40 (PB4)
- new net PB5_GPIO: U2.41 (PB5)
- new net PB8_SERVO0: U2.45 (PB8)
- new net PB9_SERVO1: U2.46 (PB9)
- new net PC13_V0: U2.2 (PC13)
- new net PC14_V1: U2.3 (PC14)
- new net PC15_V2: U2.4 (PC15)
- new net SWCLK: U2.37 (PA14)
- new net SWDIO: U2.34 (PA13)
- new net UART1_RX: U2.31 (PA10)
- new net UART1_TX: U2.30 (PA9)
- new net UART2_RX: U2.13 (PA3)
- new net UART2_TX: U2.12 (PA2)
- new net UART3_RX: U2.22 (PB11)
- new net UART3_TX: U2.21 (PB10)
- no-connect marks 0 -> 5
Other:
- note added: "~22.3V"
- note added: "~5.1A"
- moved on the sheet: C1, C10, C11, C2, C3, C4, C5, C6, C7, C8, C9, L1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

Commit message: 4/18
Parts:
- removed SW2: BOOT0, Button_Switch_SMD:SW_SPST_TL3342, symbol Switch:SW_Push
- removed Y1: 8Mhz, Crystal:Crystal_SMD_5032-2Pin_5.0x3.2mm, symbol Device:Crystal_Small
- added C28, C29, C30: 100n, Capacitor_SMD:C_0603_1608Metric, symbol Device:C_Small
- added C31: 20p, Capacitor_SMD:C_0603_1608Metric, symbol Device:C_Small
- added C32: 47u, Capacitor_Tantalum_SMD:CP_EIA-3216-18_Kemet-A_Pad1.58x1.35mm_HandSolder, symbol Device:C_Polarized_Small
- added C34, C35, C37, C40: 10u, Capacitor_SMD:C_0603_1608Metric, symbol Device:C_Small
- added C39: 10n, Capacitor_SMD:C_0603_1608Metric, symbol Device:C_Small
- added L2: 6u8, Inductor_SMD:L_Sunlord_MWSA0402S, symbol Device:L
- added R24, R25, R29: 10k, Resistor_SMD:R_0603_1608Metric, symbol Device:R_Small
- added R26: 330R, Resistor_SMD:R_0603_1608Metric, symbol Device:R_Small
- added R27: 1k, Resistor_SMD:R_0603_1608Metric, symbol Device:R_Small
- added R28: 54k6, Resistor_SMD:R_0603_1608Metric, symbol Device:R_Small
- added SW5: BTN, Button_Switch_SMD:SW_SPST_PTS810, symbol Switch:SW_Push
- added U4: RY8411, Package_TO_SOT_SMD:SOT-23-6, symbol RM24:SY8301
- added U5: RS3236, Package_TO_SOT_SMD:SOT-23-5, symbol Regulator_Linear:LDK130-12_SOT23_SOT353
- added Y2: 8Mhz, Crystal:Crystal_SMD_3225-4Pin_3.2x2.5mm, symbol Device:Crystal_GND24_Small
- C20: value 100n -> 10u; footprint Capacitor_SMD:C_0603_1608Metric -> Capacitor_SMD:C_1206_3216Metric
- C21: value 4.7u -> 10u; footprint Capacitor_SMD:C_0603_1608Metric -> Capacitor_SMD:C_1206_3216Metric
- J1: footprint (none) -> Connector_USB:USB_C_Receptacle_Palconn_UTC16-G
- R13: value 47k -> 1M
- R17: value 330R -> 10k
- R18: value 10k -> 1k
- SW1: value RST -> BTN; footprint Button_Switch_SMD:SW_SPST_TL3342 -> Button_Switch_SMD:SW_SPST_PTS810
Connections:
- net +3V3: now also C22.1, C23.1, C24.1, C25.1, C26.1, U2.1 (VBAT), U2.24 (VDD), U2.36 (VDD), U2.48 (VDD), U2.9 (VDDA), C40.1, R25.2, U5.5 (OUT)
- net BOOT0: now also R24.1; no longer C20.1, R17.1
- net GND: now also R18.2, C29.2, C30.2, C32.2, C34.2, C35.2, C37.2, C39.2, C40.2, R24.2, R27.2, R29.2, SW5.2, U4.2 (GND), U5.2 (GND), Y2.2, Y2.4; no longer R19.2
- net NRST: now also C29.1, R25.1; no longer C19.1, R16.1
- net PB0_LED0: no longer U2.18 (PB0)
- net PB1_LED1: no longer U2.19 (PB1)
- net PB2_LED2: no longer U2.20 (PB2)
- net VIN: now also C20.1, C21.1, R1.1, R17.1, U4.4 (EN), U4.5 (IN)
- net VINP: no longer R1.1
- net VOUT: now also R19.1
- net at C17.2, U2.5 (PD0): now also Y2.3
- net at C18.2, U2.6 (PD1): now also Y2.1
- net VS_VIN: now reaches R17.2
- net VS_VIN: now also R18.1; no longer R19.1
- net at R16.2, SW1.1: no longer R18.2
- removed net +3.3V: C21.1, C22.1, C23.1, C24.1, C25.1, C26.1, R18.1, U2.1 (VBAT), U2.24 (VDD), U2.36 (VDD), U2.48 (VDD), U2.9 (VDDA)
- net CAN_RX: no longer names the net of U2.32 (PA11)
- net CAN_TX: no longer names the net of U2.33 (PA12)
- net I2C1_SCL: no longer names the net of U2.42 (PB6)
- net I2C1_SDA: no longer names the net of U2.43 (PB7)
- net PA0_GPIO: no longer names the net of U2.10 (PA0)
- net PA15_GPIO: no longer names the net of U2.38 (PA15)
- net PA1_GPIO: no longer names the net of U2.11 (PA1)
- net PA4_GPIO: no longer names the net of U2.14 (PA4)
- net PA5_GPIO: no longer names the net of U2.15 (PA5)
- net PA6_GPIO: no longer names the net of U2.16 (PA6)
- net PA7_GPIO: no longer names the net of U2.17 (PA7)
- net PA8_BUZZER: no longer names the net of U2.29 (PA8)
- net PB12_GPIO: no longer names the net of U2.25 (PB12)
- net PB13_GPIO: no longer names the net of U2.26 (PB13)
- net PB14_GPIO: no longer names the net of U2.27 (PB14)
- net PB15_GPIO: no longer names the net of U2.28 (PB15)
- net PB3_GPIO: no longer names the net of U2.39 (PB3)
- net PB4_GPIO: no longer names the net of U2.40 (PB4)
- net PB5_GPIO: no longer names the net of U2.41 (PB5)
- net PB8_SERVO0: no longer names the net of U2.45 (PB8)
- net PB9_SERVO1: no longer names the net of U2.46 (PB9)
- net PC13_V0: no longer names the net of U2.2 (PC13)
- net PC14_V1: no longer names the net of U2.3 (PC14)
- net PC15_V2: no longer names the net of U2.4 (PC15)
- net UART1_RX: no longer names the net of U2.31 (PA10)
- net UART1_TX: no longer names the net of U2.30 (PA9)
- net UART2_RX: no longer names the net of U2.13 (PA3)
- net UART2_TX: no longer names the net of U2.12 (PA2)
- net UART3_RX: no longer names the net of U2.22 (PB11)
- net UART3_TX: no longer names the net of U2.21 (PB10)
- new net: R26.2, SW5.1
- new net: C31.2, R28.2, R29.1, U4.3 (FB)
- new net: C39.1, U5.4 (BP)
- new net: C28.1, U4.1 (BS)
- new net: C28.2, L2.1, U4.6 (LX)
- new net +5V: C31.1, C32.1, C34.1, C35.1, C37.1, L2.2, R28.1, U5.1 (IN), U5.3 (EN)
- new net BTN1: C30.1, R26.1
- new net BTN2: C19.1, R16.1
- new net VS_VOUT: R19.2, R27.1
Other:
- note added: "Shoule be around 5.2V"
- moved on the sheet: C1, C10, C11, C13, C14, C15, C16, C17, C18, C2, C22, C23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
